File: i2c-LevelShifter.sch (KiCad schematic (older format))
At the start: 0 parts

Commit message: Added new part and created initial schematic
Parts:
- added Q? (x2): FDC6305N, SOT-6, symbol FDC6305N
- added R? (x4): R, symbol R
Connections:
- net labels added: SCL1, SCL2, SDA1, SDA2, Vdd1, Vdd2
- wire segments 0 -> 19
Changed lines of the file:
@@
 LIBS:contrib
 LIBS:valves
-EELAYER 27 0
+LIBS:LevelShifter Components
+LIBS:i2c-LevelShifter-cache
+EELAYER 25 0
 EELAYER END
 $Descr A4 11693 8268
@@
 Comment4 ""
 $EndDescr
+$Comp
+L FDC6305N Q?
+U 1 1 54FFE888
+P 4850 2650
+F 0 "Q?" V 5050 2700 40  0000 R CNN
+F 1 "FDC6305N" V 5050 2800 40  0001 R CNN
+F 2 "SOT-6" H 4720 2752 29  0001 C CNN
+F 3 "" H 4850 2650 60  0000 C CNN
+F 4 "FDC6305N" H 4850 2650 60  0001 C CNN "MPN"
+	1    4850 2650
+	0    1    1    0
+$EndComp
+$Comp
+L FDC6305N Q?
+U 2 1 54FFE8ED
+P 5300 3300
+F 0 "Q?" V 5550 3350 40  0000 R CNN
+F 1 "FDC6305N" V 5500 3450 40  0001 R CNN
+F 2 "SOT-6" H 5170 3402 29  0001 C CNN
+F 3 "" H 5300 3300 60  0000 C CNN
+F 4 "FDC6305N" V 5300 3300 60  0001 C CNN "MPN"
+	2    5300 3300
+	0    1    1    0
+$EndComp
+Wire Wire Line
+	5250 2100 5250 3100
+Wire Wire Line
+	5100 3400 4400 3400
+Wire Wire Line
+	4400 3400 3250 3400
+Wire Wire Line
+	5500 3400 5700 3400
+Wire Wire Line
+	5700 3400 6800 3400
+Wire Wire Line
+	5050 2750 6000 2750
+Wire Wire Line
+	6000 2750 6800 2750
+Wire Wire Line
+	4650 2750 4100 2750
+Wire Wire Line
+	4100 2750 3250 2750
+$Comp
+L R R?
+U 1 1 54FFEABF
+P 4100 2350
+F 0 "R?" V 4180 2350 50  0000 C CNN
+F 1 "R" V 4107 2351 50  0000 C CNN
+F 2 "" V 4030 2350 30  0000 C CNN
+F 3 "" H 4100 2350 30  0000 C CNN
+	1    4100 2350
+	1    0    0    -1
+$EndComp
+$Comp
+L R R?
+U 1 1 54FFEB5A
+P 4400 2350
+F 0 "R?" V 4480 2350 50  0000 C CNN
+F 1 "R" V 4407 2351 50  0000 C CNN
+F 2 "" V 4330 2350 30  0000 C CNN
+F 3 "" H 4400 2350 30  0000 C CNN
+	1    4400 2350
+	1    0    0    -1
+$EndComp
+$Comp
+L R R?
+U 1 1 54FFEB90
+P 5700 2350
+F 0 "R?" V 5780 2350 50  0000 C CNN
+F 1 "R" V 5707 2351 50  0000 C CNN
+F 2 "" V 5630 2350 30  0000 C CNN
+F 3 "" H 5700 2350 30  0000 C CNN
+	1    5700 2350
+	1    0    0    -1
+$EndComp
+$Comp
+L R R?
+U 1 1 54FFEBCF
+P 6000 2350
+F 0 "R?" V 6080 2350 50  0000 C CNN
+F 1 "R" V 6007 2351 50  0000 C CNN
+F 2 "" V 5930 2350 30  0000 C CNN
+F 3 "" H 6000 2350 30  0000 C CNN
+	1    6000 2350
+	1    0    0    -1
+$EndComp
+Wire Wire Line
+	3250 2100 4100 2100
+Wire Wire Line
+	4100 2100 4400 2100
+Wire Wire Line
+	4400 2100 4800 2100
+Wire Wire Line
+	4800 2100 5250 2100
+Connection ~ 4100 2100
+Wire Wire Line
+	4800 2100 4800 2450
+Connection ~ 4400 2100
+Connection ~ 4800 2100
+Wire Wire Line
+	4400 2600 4400 3400
+Connection ~ 4400 3400
+Wire Wire Line
+	4100 2600 4100 2750
+Connection ~ 4100 2750
+Wire Wire Line
+	5700 2600 5700 3400
+Connection ~ 5700 3400
+Wire Wire Line
+	6000 2600 6000 2750
+Connection ~ 6000 2750
+Wire Wire Line
+	5700 2100 6800 2100
+Text Label 6500 2100 0    60   ~ 0
+Vdd2
+Text Label 6500 2750 0    60   ~ 0
+SDA2
+Text Label 6500 3400 0    60   ~ 0
+SCL2
+Text Label 3300 2100 0    60   ~ 0
+Vdd1
+Text Label 3300 2750 0    60   ~ 0
+SDA1
+Text Label 3300 3400 0    60   ~ 0
+SCL1
 $EndSCHEMATC

Commit message: Added connectors to the schematic
Parts:
- added P?: 5v, symbol CONN_01X03
- added P?: 3.3v, symbol CONN_01X03
- Q? (x2): ConradPN (none) -> 1263351-62
Connections:
- net labels added: Vdd1=3.3v, Vdd2=5v
- net labels removed: Vdd1, Vdd2
- wire segments 19 -> 32
Changed lines of the file:
@@
 L FDC6305N Q?
 U 1 1 54FFE888
-P 4850 2650
-F 0 "Q?" V 5050 2700 40  0000 R CNN
-F 1 "FDC6305N" V 5050 2800 40  0001 R CNN
-F 2 "SOT-6" H 4720 2752 29  0001 C CNN
-F 3 "" H 4850 2650 60  0000 C CNN
-F 4 "FDC6305N" H 4850 2650 60  0001 C CNN "MPN"
-	1    4850 2650
+P 4850 2750
+F 0 "Q?" V 5050 2800 40  0000 R CNN
+F 1 "FDC6305N" V 5050 2900 40  0001 R CNN
+F 2 "SOT-6" H 4720 2852 29  0001 C CNN
+F 3 "" H 4850 2750 60  0000 C CNN
+F 4 "FDC6305N" H 4850 2750 60  0001 C CNN "MPN"
+F 5 "1263351-62" V 4850 2750 60  0001 C CNN "ConradPN"
+	1    4850 2750
 	0    1    1    0
 $EndComp
@@
 F 3 "" H 5300 3300 60  0000 C CNN
 F 4 "FDC6305N" V 5300 3300 60  0001 C CNN "MPN"
+F 5 "1263351-62" V 5300 3300 60  0001 C CNN "ConradPN"
 	2    5300 3300
 	0    1    1    0
@@
 	5250 2100 5250 3100
 Wire Wire Line
-	5100 3400 4400 3400
+	3100 3400 4400 3400
 Wire Wire Line
-	4400 3400 3250 3400
+	4400 3400 5100 3400
 Wire Wire Line
 	5500 3400 5700 3400
 Wire Wire Line
-	5700 3400 6800 3400
+	5700 3400 6900 3400
 Wire Wire Line
-	5050 2750 6000 2750
+	5050 2850 6000 2850
 Wire Wire Line
-	6000 2750 6800 2750
+	6000 2850 6750 2850
 Wire Wire Line
-	4650 2750 4100 2750
+	3250 2850 4100 2850
 Wire Wire Line
-	4100 2750 3250 2750
+	4100 2850 4650 2850
 $Comp
 L R R?
 U 1 1 54FFEABF
-P 4100 2350
-F 0 "R?" V 4180 2350 50  0000 C CNN
-F 1 "R" V 4107 2351 50  0000 C CNN
-F 2 "" V 4030 2350 30  0000 C CNN
-F 3 "" H 4100 2350 30  0000 C CNN
-	1    4100 2350
+P 4100 2450
+F 0 "R?" V 4180 2450 50  0000 C CNN
+F 1 "R" V 4107 2451 50  0000 C CNN
+F 2 "" V 4030 2450 30  0000 C CNN
+F 3 "" H 4100 2450 30  0000 C CNN
+	1    4100 2450
 	1    0    0    -1
 $EndComp
@@
 L R R?
 U 1 1 54FFEB5A
-P 4400 2350
-F 0 "R?" V 4480 2350 50  0000 C CNN
-F 1 "R" V 4407 2351 50  0000 C CNN
-F 2 "" V 4330 2350 30  0000 C CNN
-F 3 "" H 4400 2350 30  0000 C CNN
-	1    4400 2350
+P 4400 2450
+F 0 "R?" V 4480 2450 50  0000 C CNN
+F 1 "R" V 4407 2451 50  0000 C CNN
+F 2 "" V 4330 2450 30  0000 C CNN
+F 3 "" H 4400 2450 30  0000 C CNN
+	1    4400 2450
 	1    0    0    -1
 $EndComp
@@
 L R R?
 U 1 1 54FFEB90
-P 5700 2350
-F 0 "R?" V 5780 2350 50  0000 C CNN
-F 1 "R" V 5707 2351 50  0000 C CNN
-F 2 "" V 5630 2350 30  0000 C CNN
-F 3 "" H 5700 2350 30  0000 C CNN
-	1    5700 2350
+P 5700 2450
+F 0 "R?" V 5780 2450 50  0000 C CNN
+F 1 "R" V 5707 2451 50  0000 C CNN
+F 2 "" V 5630 2450 30  0000 C CNN
+F 3 "" H 5700 2450 30  0000 C CNN
+	1    5700 2450
 	1    0    0    -1
 $EndComp
@@
 L R R?
 U 1 1 54FFEBCF
-P 6000 2350
-F 0 "R?" V 6080 2350 50  0000 C CNN
-F 1 "R" V 6007 2351 50  0000 C CNN
-F 2 "" V 5930 2350 30  0000 C CNN
-F 3 "" H 6000 2350 30  0000 C CNN
-	1    6000 2350
+P 6000 2450
+F 0 "R?" V 6080 2450 50  0000 C CNN
+F 1 "R" V 6007 2451 50  0000 C CNN
+F 2 "" V 5930 2450 30  0000 C CNN
+F 3 "" H 6000 2450 30  0000 C CNN
+	1    6000 2450
 	1    0    0    -1
 $EndComp
 Wire Wire Line
-	3250 2100 4100 2100
+	2850 2100 4100 2100
 Wire Wire Line
 	4100 2100 4400 2100
@@
 Connection ~ 4100 2100
 Wire Wire Line
-	4800 2100 4800 2450
+	4800 2100 4800 2550
 Connection ~ 4400 2100
 Connection ~ 4800 2100
 Wire Wire Line
-	4400 2600 4400 3400
+	4400 2700 4400 3400
 Connection ~ 4400 3400
 Wire Wire Line
-	4100 2600 4100 2750
-Connection ~ 4100 2750
+	4100 2600 4100 2850
+Connection ~ 4100 2850
 Wire Wire Line
-	5700 2600 5700 3400
+	5700 2700 5700 3400
 Connection ~ 5700 3400
 Wire Wire Line
-	6000 2600 6000 2750
-Connection ~ 6000 2750
+	6000 2700 6000 2850
+Connection ~ 6000 2850
 Wire Wire Line
-	5700 2100 6800 2100
-Text Label 6500 2100 0    60   ~ 0
-Vdd2
-Text Label 6500 2750 0    60   ~ 0
+	5700 2100 6000 2100
+Wire Wire Line
+	6000 2100 7150 2100
+Text Label 6350 2100 0    60   ~ 0
+Vdd2=5v
+Text Label 6350 2850 0    60   ~ 0
 SDA2
 Text Label 6500 3400 0    60   ~ 0
 SCL2
 Text Label 3300 2100 0    60   ~ 0
-Vdd1
-Text Label 3300 2750 0    60   ~ 0
+Vdd1=3.3v
+Text Label 3400 2850 0    60   ~ 0
 SDA1
 Text Label 3300 3400 0    60   ~ 0
 SCL1
+$Comp
+L CONN_01X03 P?
+U 1 1 55002841
+P 7350 2200
+F 0 "P?" H 7350 2000 50  0000 C CNN
+F 1 "5v" H 7350 2400 50  0000 C CNN
+F 2 "" H 7350 2200 60  0000 C CNN
+F 3 "" H 7350 2200 60  0000 C CNN
+F 4 "1945106" H 7350 2200 60  0001 C CNN "MPN"
+F 5 "744336-62 " H 7350 2200 60  0001 C CNN "ConradPN"
+	1    7350 2200
+	1    0    0    -1
+$EndComp
+$Comp
+L CONN_01X03 P?
+U 1 1 5500287E
+P 2650 2200
+F 0 "P?" H 2650 2400 50  0000 C CNN
+F 1 "3.3v" H 2650 2000 50  0000 C CNN
+F 2 "" H 2650 2200 60  0000 C CNN
+F 3 "" H 2650 2200 60  0000 C CNN
+F 4 "1945106" H 2650 2200 60  0001 C CNN "MPN"
+F 5 "744336-62 " H 2650 2200 60  0001 C CNN "ConradPN"
+	1    2650 2200
+	-1   0    0    1
+$EndComp
+Wire Wire Line
+	6750 2850 6750 2200
+Wire Wire Line
+	6750 2200 7150 2200
+Wire Wire Line
+	6900 3400 6900 2300
+Wire Wire Line
+	6900 2300 7150 2300
+Wire Wire Line
+	3250 2850 3250 2200
+Wire Wire Line
+	3250 2200 2850 2200
+Wire Wire Line
+	3100 3400 3100 2300
+Wire Wire Line
+	3100 2300 2850 2300
+Wire Wire Line
+	5700 2100 5700 2200
+Wire Wire Line
+	6000 2100 6000 2200
+Connection ~ 6000 2100
+Wire Wire Line
+	4100 2100 4100 2200
+Wire Wire Line
+	4400 2100 4400 2200
 $EndSCHEMATC

Commit message: Added ltspice model and annotated the schema with the calculations
Parts:
- removed P?: 5v, symbol CONN_01X03
- removed P?: 3.3v, symbol CONN_01X03
- removed Q? (x2): FDC6305N, SOT-6, symbol FDC6305N
- added P101, P103: 3v3, symbol CONN_01X02
- added P102, P104: 5v, symbol CONN_01X02
- added Q101, Q102: IRLML2502, Micro3, symbol IRLML2502
- R101, R102: renamed from R?; value R -> 10k
- R103, R104: renamed from R?; value R -> 1k5
Connections:
- net labels added: GND, VDD1=3v3, VDD2=5v, VSS2=5v
- net labels removed: Vdd1=3.3v, Vdd2=5v
Other:
- note added: "When SDA1 goes low, the voltage across Q101 gs \nwill be 3.3V which is higher than the threshold \nvoltage of 1.2V, so Q101 ds will start to conduct \nthrough R104.\n\n R104 = 1k5\n VDD2 = 5v\n Vgs(th) = 1.2V\n \n Ir104 = VDD2 : R104\n Ir104 = 5 : 1k5\n Ir104 = 3.333... mA\n\nThe selected part has an Id of 4.2 A\n\nThis implies a high impedence of the device(s)\nconnected to the SDA1."
Changed lines of the file:
@@
 $EndDescr
 $Comp
-L FDC6305N Q?
-U 1 1 54FFE888
-P 4850 2750
-F 0 "Q?" V 5050 2800 40  0000 R CNN
-F 1 "FDC6305N" V 5050 2900 40  0001 R CNN
-F 2 "SOT-6" H 4720 2852 29  0001 C CNN
-F 3 "" H 4850 2750 60  0000 C CNN
-F 4 "FDC6305N" H 4850 2750 60  0001 C CNN "MPN"
-F 5 "1263351-62" V 4850 2750 60  0001 C CNN "ConradPN"
-	1    4850 2750
-	0    1    1    0
-$EndComp
-$Comp
-L FDC6305N Q?
-U 2 1 54FFE8ED
-P 5300 3300
-F 0 "Q?" V 5550 3350 40  0000 R CNN
-F 1 "FDC6305N" V 5500 3450 40  0001 R CNN
-F 2 "SOT-6" H 5170 3402 29  0001 C CNN
-F 3 "" H 5300 3300 60  0000 C CNN
-F 4 "FDC6305N" V 5300 3300 60  0001 C CNN "MPN"
-F 5 "1263351-62" V 5300 3300 60  0001 C CNN "ConradPN"
-	2    5300 3300
-	0    1    1    0
-$EndComp
-Wire Wire Line
-	5250 2100 5250 3100
-Wire Wire Line
-	3100 3400 4400 3400
-Wire Wire Line
-	4400 3400 5100 3400
-Wire Wire Line
-	5500 3400 5700 3400
-Wire Wire Line
-	5700 3400 6900 3400
-Wire Wire Line
-	5050 2850 6000 2850
-Wire Wire Line
-	6000 2850 6750 2850
-Wire Wire Line
-	3250 2850 4100 2850
-Wire Wire Line
-	4100 2850 4650 2850
-$Comp
-L R R?
+L R R101
 U 1 1 54FFEABF
 P 4100 2450
-F 0 "R?" V 4180 2450 50  0000 C CNN
-F 1 "R" V 4107 2451 50  0000 C CNN
+F 0 "R101" H 4250 2450 50  0000 C CNN
+F 1 "10k" V 4107 2451 50  0000 C CNN
 F 2 "" V 4030 2450 30  0000 C CNN
 F 3 "" H 4100 2450 30  0000 C CNN
@@
 $EndComp
 $Comp
-L R R?
+L R R102
 U 1 1 54FFEB5A
 P 4400 2450
-F 0 "R?" V 4480 2450 50  0000 C CNN
-F 1 "R" V 4407 2451 50  0000 C CNN
+F 0 "R102" H 4550 2450 50  0000 C CNN
+F 1 "10k" V 4407 2451 50  0000 C CNN
 F 2 "" V 4330 2450 30  0000 C CNN
 F 3 "" H 4400 2450 30  0000 C CNN
@@
 $EndComp
 $Comp
-L R R?
+L R R103
 U 1 1 54FFEB90
 P 5700 2450
-F 0 "R?" V 5780 2450 50  0000 C CNN
-F 1 "R" V 5707 2451 50  0000 C CNN
+F 0 "R103" H 5850 2450 50  0000 C CNN
+F 1 "1k5" V 5707 2451 50  0000 C CNN
 F 2 "" V 5630 2450 30  0000 C CNN
 F 3 "" H 5700 2450 30  0000 C CNN
@@
 $EndComp
 $Comp
-L R R?
+L R R104
 U 1 1 54FFEBCF
 P 6000 2450
-F 0 "R?" V 6080 2450 50  0000 C CNN
-F 1 "R" V 6007 2451 50  0000 C CNN
+F 0 "R104" H 6150 2450 50  0000 C CNN
+F 1 "1k5" V 6007 2451 50  0000 C CNN
 F 2 "" V 5930 2450 30  0000 C CNN
 F 3 "" H 6000 2450 30  0000 C CNN
@@
 	1    0    0    -1
 $EndComp
-Wire Wire Line
-	2850 2100 4100 2100
+Text Label 6450 2100 0    60   ~ 0
+VDD2=5v
+Text Label 6550 2850 0    60   ~ 0
+SDA2
+Text Label 6600 3400 0    60   ~ 0
+SCL2
+Text Label 3500 2100 0    60   ~ 0
+VDD1=3v3
+Text Label 3550 2850 0    60   ~ 0
+SDA1
+Text Label 3500 3400 0    60   ~ 0
+SCL1
+$Comp
+L CONN_01X02 P101
+U 1 1 55009AA3
+P 4000 1100
+F 0 "P101" H 4000 1250 50  0000 C CNN
+F 1 "3v3" H 4000 950 50  0000 C CNN
+F 2 "" H 4000 1100 60  0000 C CNN
+F 3 "" H 4000 1100 60  0000 C CNN
+	1    4000 1100
+	1    0    0    -1
+$EndComp
+$Comp
+L CONN_01X02 P102
+U 1 1 55009B79
+P 6200 1100
+F 0 "P102" H 6200 950 50  0000 C CNN
+F 1 "5v" H 6200 1250 50  0000 C CNN
+F 2 "" H 6200 1100 60  0000 C CNN
+F 3 "" H 6200 1100 60  0000 C CNN
+	1    6200 1100
+	-1   0    0    1
+$EndComp
+Wire Wire Line
+	5250 2100 5250 3100
+Wire Wire Line
+	3350 3400 4400 3400
+Wire Wire Line
+	4400 3400 5100 3400
+Wire Wire Line
+	5500 3400 5700 3400
+Wire Wire Line
+	5700 3400 6900 3400
+Wire Wire Line
+	5050 2850 6000 2850
+Wire Wire Line
+	6000 2850 6900 2850
+Wire Wire Line
+	3350 2850 4100 2850
+Wire Wire Line
+	4100 2850 4650 2850
+Wire Wire Line
+	3350 2100 4100 2100
 Wire Wire Line
 	4100 2100 4400 2100
@@
 Connection ~ 4100 2850
 Wire Wire Line
-	5700 2700 5700 3400
+	5700 3400 5700 2700
 Connection ~ 5700 3400
 Wire Wire Line
@@
 	5700 2100 6000 2100
 Wire Wire Line
-	6000 2100 7150 2100
-Text Label 6350 2100 0    60   ~ 0
-Vdd2=5v
-Text Label 6350 2850 0    60   ~ 0
-SDA2
-Text Label 6500 3400 0    60   ~ 0
-SCL2
-Text Label 3300 2100 0    60   ~ 0
-Vdd1=3.3v
-Text Label 3400 2850 0    60   ~ 0
-SDA1
-Text Label 3300 3400 0    60   ~ 0
-SCL1
-$Comp
-L CONN_01X03 P?
-U 1 1 55002841
-P 7350 2200
-F 0 "P?" H 7350 2000 50  0000 C CNN
-F 1 "5v" H 7350 2400 50  0000 C CNN
-F 2 "" H 7350 2200 60  0000 C CNN
-F 3 "" H 7350 2200 60  0000 C CNN
-F 4 "1945106" H 7350 2200 60  0001 C CNN "MPN"
-F 5 "744336-62 " H 7350 2200 60  0001 C CNN "ConradPN"
-	1    7350 2200
-	1    0    0    -1
-$EndComp
-$Comp
-L CONN_01X03 P?
-U 1 1 5500287E
-P 2650 2200
-F 0 "P?" H 2650 2400 50  0000 C CNN
-F 1 "3.3v" H 2650 2000 50  0000 C CNN
-F 2 "" H 2650 2200 60  0000 C CNN
-F 3 "" H 2650 2200 60  0000 C CNN
-F 4 "1945106" H 2650 2200 60  0001 C CNN "MPN"
-F 5 "744336-62 " H 2650 2200 60  0001 C CNN "ConradPN"
-	1    2650 2200
-	-1   0    0    1
-$EndComp
-Wire Wire Line
-	6750 2850 6750 2200
-Wire Wire Line
-	6750 2200 7150 2200
-Wire Wire Line
-	6900 3400 6900 2300
-Wire Wire Line
-	6900 2300 7150 2300
-Wire Wire Line
-	3250 2850 3250 2200
-Wire Wire Line
-	3250 2200 2850 2200
-Wire Wire Line
-	3100 3400 3100 2300
-Wire Wire Line
-	3100 2300 2850 2300
+	6000 2100 6950 2100
 Wire Wire Line
 	5700 2100 5700 2200
@@
 Wire Wire Line
 	4400 2100 4400 2200
+Wire Wire Line
+	3800 1050 3250 1050
+Wire Wire Line
+	3800 1150 3600 1150
+Wire Wire Line
+	3600 1150 3600 1450
+$Comp
+L GND #PWR102
+U 1 1 55009C82
+P 3600 1450
+F 0 "#PWR102" H 3600 1200 60  0001 C CNN
+F 1 "GND" H 3600 1300 60  0000 C CNN
+F 2 "" H 3600 1450 60  0000 C CNN
+F 3 "" H 3600 1450 60  0000 C CNN
+	1    3600 1450
+	1    0    0    -1
+$EndComp
+Text Label 3300 1050 0    60   ~ 0
+VDD1=3v3
+Wire Wire Line
+	6400 1150 6700 1150
+Wire Wire Line
+	6700 1150 6700 1400
+Wire Wire Line
+	6400 1050 7050 1050
+Text Label 6550 1050 0    60   ~ 0
+VSS2=5v
+$Comp
+L GND #PWR101
+U 1 1 55009D67
+P 6700 1400
+F 0 "#PWR101" H 6700 1150 60  0001 C CNN
+F 1 "GND" H 6700 1250 60  0000 C CNN
+F 2 "" H 6700 1400 60  0000 C CNN
+F 3 "" H 6700 1400 60  0000 C CNN
+	1    6700 1400
+	1    0    0    -1
+$EndComp
+$Comp
+L CONN_01X02 P103
+U 1 1 5500A304
+P 3150 2900
+F 0 "P103" H 3150 3050 50  0000 C CNN
+F 1 "3v3" H 3150 2750 50  0000 C CNN
+F 2 "" H 3150 2900 60  0000 C CNN
+F 3 "" H 3150 2900 60  0000 C CNN
+	1    3150 2900
+	-1   0    0    1
+$EndComp
+$Comp
+L CONN_01X02 P104
+U 1 1 5500A353
+P 7100 2900
+F 0 "P104" H 7100 2750 50  0000 C CNN
+F 1 "5v" H 7100 3050 50  0000 C CNN
+F 2 "" H 7100 2900 60  0000 C CNN
+F 3 "" H 7100 2900 60  0000 C CNN
+	1    7100 2900
+	1    0    0    -1
+$EndComp
+Wire Wire Line
+	6900 3400 6900 2950
+Wire Wire Line
+	3350 3400 3350 2950
+$Comp
+L IRLML2502 Q101
+U 1 1 5500B552
+P 4850 2750
+F 0 "Q101" V 4750 2950 40  0000 R CNN
+F 1 "IRLML2502" V 5100 2850 40  0000 R CNN
+F 2 "Micro3" H 4720 2852 29  0001 C CNN
+F 3 "" H 4850 2750 60  0000 C CNN
+	1    4850 2750
+	0    1    1    0
+$EndComp
+$Comp
+L IRLML2502 Q102
+U 1 1 5500B5B3
+P 5300 3300
+F 0 "Q102" V 5200 3500 40  0000 R CNN
+F 1 "IRLML2502" V 5550 3450 40  0000 R CNN
+F 2 "Micro3" H 5170 3402 29  0001 C CNN
+F 3 "" H 5300 3300 60  0000 C CNN
+	1    5300 3300
+	0    1    1    0
+$EndComp
+Text Notes 3000 5200 0    60   ~ 0
+When SDA1 goes low, the voltage across Q101 gs \nwill be 3.3V which is higher than the threshold \nvoltage of 1.2V, so Q101 ds will start to conduct \nthrough R104.\n\n	R104 = 1k5\n	VDD2 = 5v\n	Vgs(th) = 1.2V\n \n	Ir104 = VDD2 : R104\n	Ir104 = 5 : 1k5\n	Ir104 = 3.333... mA\n\nThe selected part has an Id of 4.2 A\n\nThis implies a high impedence of the device(s)\nconnected to the SDA1.
 $EndSCHEMATC

Commit message: Added MPN to the template field names
Connections:
- net labels removed: VDD2=5v
- wire segments 32 -> 20
Other:
- note added: "When SDA1 is pulled low, the voltage across \nQ101 gs will be 3.3V which is higher than the \nthreshold voltage of 1.2V, so Q101 ds will \nstart to conduct through R104.\n\n R104 = 1k5\n VDD2 = 5v\n Vgs(th) = 1.2V\n \n Ir104 = VDD2 : R104\n Ir104 = 5 : 1k5\n Ir104 = 3.333... mA\n\nThe selected part has an Id of 4.2 A\n\nThis implies a high impedence of the device(s)\nconnected to the SDA1."
- note removed: "When SDA1 goes low, the voltage across Q101 gs \nwill be 3.3V which is higher than the threshold \nvoltage of 1.2V, so Q101 ds will start to conduct \nthrough R104.\n\n R104 = 1k5\n VDD2 = 5v\n Vgs(th) = 1.2V\n \n Ir104 = VDD2 : R104\n Ir104 = 5 : 1k5\n Ir104 = 3.333... mA\n\nThe selected part has an Id of 4.2 A\n\nThis implies a high impedence of the device(s)\nconnected to the SDA1."

Commit message: Completed layout and Gerber files
Parts:
- removed P101, P103: 3v3, symbol CONN_01X02
- removed P102, P104: 5v, symbol CONN_01X02
- added P101: 3v3, Socket_Strips:Socket_Strip_Straight_1x04, symbol CONN_01X04
- added P102: 5v, Socket_Strips:Socket_Strip_Straight_1x04, symbol CONN_01X04
- Q101, Q102: footprint Micro3 -> i2cLib:Micro3; ConradPN (none) -> 162827 - 62; MPN (none) -> IRLML2502TRPBF
- R101, R102, R103, R104: footprint (none) -> Resistors_SMD:R_0805
Connections:
- wire segments 20 -> 26
Changed lines of the file:
@@
 F 0 "R101" H 4850 1950 50  0000 C CNN
 F 1 "10k" V 4707 1951 50  0000 C CNN
-F 2 "" V 4630 1950 30  0000 C CNN
+F 2 "Resistors_SMD:R_0805" V 4630 1950 30  0001 C CNN
 F 3 "" H 4700 1950 30  0000 C CNN
 	1    4700 1950
@@
 F 0 "R102" H 5150 1950 50  0000 C CNN
 F 1 "10k" V 5007 1951 50  0000 C CNN
-F 2 "" V 4930 1950 30  0000 C CNN
+F 2 "Resistors_SMD:R_0805" V 4930 1950 30  0001 C CNN
 F 3 "" H 5000 1950 30  0000 C CNN
 	1    5000 1950
@@
 F 0 "R103" H 6450 1950 50  0000 C CNN
 F 1 "1k5" V 6307 1951 50  0000 C CNN
-F 2 "" V 6230 1950 30  0000 C CNN
+F 2 "Resistors_SMD:R_0805" V 6230 1950 30  0001 C CNN
 F 3 "" H 6300 1950 30  0000 C CNN
 	1    6300 1950
@@
 F 0 "R104" H 6750 1950 50  0000 C CNN
 F 1 "1k5" V 6607 1951 50  0000 C CNN
-F 2 "" V 6530 1950 30  0000 C CNN
+F 2 "Resistors_SMD:R_0805" V 6530 1950 30  0001 C CNN
 F 3 "" H 6600 1950 30  0000 C CNN
 	1    6600 1950
@@
 Text Label 4100 2900 0    60   ~ 0
 SCL1
-$Comp
-L CONN_01X02 P101
-U 1 1 55009AA3
-P 3750 1650
-F 0 "P101" H 3750 1500 50  0000 C CNN
-F 1 "3v3" H 3750 1800 50  0000 C CNN
-F 2 "" H 3750 1650 60  0000 C CNN
-F 3 "" H 3750 1650 60  0000 C CNN
-	1    3750 1650
-	-1   0    0    -1
-$EndComp
-$Comp
-L CONN_01X02 P102
-U 1 1 55009B79
-P 7700 1650
-F 0 "P102" H 7700 1500 50  0000 C CNN
-F 1 "5v" H 7700 1800 50  0000 C CNN
-F 2 "" H 7700 1650 60  0000 C CNN
-F 3 "" H 7700 1650 60  0000 C CNN
-	1    7700 1650
-	1    0    0    -1
-$EndComp
 Wire Wire Line
 	5850 1600 5850 2600
 Wire Wire Line
-	3950 2900 5700 2900
+	3650 2900 5700 2900
 Wire Wire Line
-	6100 2900 7500 2900
+	7900 2900 6100 2900
 Wire Wire Line
-	5650 2350 7500 2350
+	5650 2350 7700 2350
 Wire Wire Line
-	3950 2350 5250 2350
+	3800 2350 5250 2350
 Wire Wire Line
-	3950 1600 5850 1600
+	3650 1600 5850 1600
 Connection ~ 4700 1600
 Wire Wire Line
@@
 Connection ~ 6600 2350
 Wire Wire Line
-	6300 1600 7500 1600
+	6300 1600 7900 1600
 Wire Wire Line
 	6300 1600 6300 1700
@@
 	1    0    0    -1
 $EndComp
-$Comp
-L CONN_01X02 P103
-U 1 1 5500A304
-P 3750 2400
-F 0 "P103" H 3750 2550 50  0000 C CNN
-F 1 "3v3" H 3750 2250 50  0000 C CNN
-F 2 "" H 3750 2400 60  0000 C CNN
-F 3 "" H 3750 2400 60  0000 C CNN
-	1    3750 2400
-	-1   0    0    1
-$EndComp
-$Comp
-L CONN_01X02 P104
-U 1 1 5500A353
-P 7700 2400
-F 0 "P104" H 7700 2250 50  0000 C CNN
-F 1 "5v" H 7700 2550 50  0000 C CNN
-F 2 "" H 7700 2400 60  0000 C CNN
-F 3 "" H 7700 2400 60  0000 C CNN
-	1    7700 2400
-	1    0    0    -1
-$EndComp
 Wire Wire Line
-	7500 2900 7500 2450
+	7900 1900 7900 2900
 Wire Wire Line
-	3950 2900 3950 2450
+	3650 1900 3650 2900
 $Comp
 L IRLML2502 Q101
@@
 F 0 "Q101" V 5350 2450 40  0000 R CNN
 F 1 "IRLML2502" V 5700 2350 40  0000 R CNN
-F 2 "Micro3" H 5320 2352 29  0001 C CNN
+F 2 "i2cLib:Micro3" H 5320 2352 29  0001 C CNN
 F 3 "" H 5450 2250 60  0000 C CNN
+F 4 "IRLML2502TRPBF" H 5450 2250 60  0001 C CNN "MPN"
+F 5 "162827 - 62" H 5450 2250 60  0001 C CNN "ConradPN"
 	1    5450 2250
 	0    1    1    0
@@
 F 0 "Q102" V 5800 3000 40  0000 R CNN
 F 1 "IRLML2502" V 6150 2950 40  0000 R CNN
-F 2 "Micro3" H 5770 2902 29  0001 C CNN
+F 2 "i2cLib:Micro3" H 5770 2902 29  0001 C CNN
 F 3 "" H 5900 2800 60  0000 C CNN
+F 4 "IRLML2502TRPBF" H 5900 2800 60  0001 C CNN "MPN"
+F 5 "162827 - 62" H 5900 2800 60  0001 C CNN "ConradPN"
 	1    5900 2800
 	0    1    1    0
@@
 Wire Wire Line
 	3950 1700 3950 1850
+$Comp
+L CONN_01X04 P101
+U 1 1 5506CE8C
+P 3450 1750
+F 0 "P101" H 3450 1450 50  0000 C CNN
+F 1 "3v3" H 3450 2000 50  0000 C CNN
+F 2 "Socket_Strips:Socket_Strip_Straight_1x04" H 3450 1750 60  0001 C CNN
+F 3 "" H 3450 1750 60  0000 C CNN
+F 4 "SCS4AA3" H 3450 1750 60  0001 C CNN "MPN"
+F 5 "1311448 - 62 " H 3450 1750 60  0001 C CNN "ConradPN"
+	1    3450 1750
+	-1   0    0    -1
+$EndComp
+Wire Wire Line
+	3650 1700 3950 1700
+Wire Wire Line
+	3800 2350 3800 1800
+Wire Wire Line
+	3800 1800 3650 1800
+$Comp
+L CONN_01X04 P102
+U 1 1 5506D0B1
+P 8100 1750
+F 0 "P102" H 8100 1450 50  0000 C CNN
+F 1 "5v" H 8100 2000 50  0000 C CNN
+F 2 "Socket_Strips:Socket_Strip_Straight_1x04" H 8100 1750 60  0001 C CNN
+F 3 "" H 8100 1750 60  0000 C CNN
+F 4 "SCS4AA3" H 8100 1750 60  0001 C CNN "MPN"
+F 5 "1311448 - 62 " H 8100 1750 60  0001 C CNN "ConradPN"
+	1    8100 1750
+	1    0    0    -1
+$EndComp
+Wire Wire Line
+	7500 1700 7900 1700
+Wire Wire Line
+	7700 2350 7700 1800
+Wire Wire Line
+	7700 1800 7900 1800
 $EndSCHEMATC
