File: i2c-LevelShifter.sch (KiCad schematic (older format))
At the start: 8 parts, among them P101 3v3, P102 5v, Q101 IRLML2502, Q102 IRLML2502

Commit message: New board layout and kiCad logo
Parts:
- Q101, Q102: footprint i2cLib:Micro3 -> SOT-23
Changed lines of the file:
@@
 LIBS:valves
 LIBS:LevelShifter Components
-LIBS:i2c-LevelShifter-cache
 EELAYER 25 0
 EELAYER END
@@
 F 0 "Q101" V 5350 2450 40  0000 R CNN
 F 1 "IRLML2502" V 5700 2350 40  0000 R CNN
-F 2 "i2cLib:Micro3" H 5320 2352 29  0001 C CNN
+F 2 "SOT-23" H 5320 2352 29  0001 C CNN
 F 3 "" H 5450 2250 60  0000 C CNN
 F 4 "IRLML2502TRPBF" H 5450 2250 60  0001 C CNN "MPN"
@@
 F 0 "Q102" V 5800 3000 40  0000 R CNN
 F 1 "IRLML2502" V 6150 2950 40  0000 R CNN
-F 2 "i2cLib:Micro3" H 5770 2902 29  0001 C CNN
+F 2 "SOT-23" H 5770 2902 29  0001 C CNN
 F 3 "" H 5900 2800 60  0000 C CNN
 F 4 "IRLML2502TRPBF" H 5900 2800 60  0001 C CNN "MPN"
